File: MiniProj.sch (KiCad schematic (older format))
At the start: 23 parts, among them SW1_UP1 SW_Push_Dual, SW2_DOWN1 SW_Push_Dual, SW3_LEFT1 SW_Push_Dual, SW4_RIGHT1 SW_Push_Dual, SW5_RESET1 SW_Push_Dual, U1 STM32F051R8Tx

Commit message: PLPCB
Rev 1
Parts:
- removed PS?: IA0305S, Converter_DCDC:Converter_DCDC_XP_POWER-IAxxxxS_THT, symbol Converter_DCDC:IA0305S
- added C8: 1uF, Capacitor_SMD:C_0402_1005Metric, symbol Device:C
- added J1: 1935161, digikey-footprints:Terminal_Block_D1.3mm_P5mm, symbol dk_Terminal-Blocks-Wire-to-Board:1935161
- added J2, J3, J4, J5: Conn_01x16_Male, Connector_PinHeader_2.54mm:PinHeader_1x16_P2.54mm_Vertical, symbol Connector:Conn_01x16_Male
- added PS1: IA0503S_copy, PDS1-S3-S3-M_1:CONV_PDS1-S3-S3-M, symbol dk_DC-DC-Converters:IA0503S_copy
- added R10: 10k, Resistor_SMD:R_0402_1005Metric, symbol Device:R
- added R11: 510, Resistor_SMD:R_0402_1005Metric, symbol Device:R
- C1, C2, C3, C4, C6, C7: footprint Capacitor_SMD:C_0201_0603Metric -> Capacitor_SMD:C_0402_1005Metric
Connections:
- net labels added: +5V, GNDREF
- net labels removed: +3V0
- wire segments 135 -> 210

Commit message: BIgger pads
Change R and C
Parts:
- C1, C2, C3, C4, C5, C6, C7, C8: footprint Capacitor_SMD:C_0402_1005Metric -> Capacitor_SMD:C_0805_2012Metric_Pad1.15x1.40mm_HandSolder
- R1, R10, R11, R2, R3, R4, R5, R6, R7, R8, R9: footprint Resistor_SMD:R_0402_1005Metric -> Resistor_SMD:R_0805_2012Metric_Pad1.15x1.40mm_HandSolder
Changed lines of the file:
@@
 F 0 "C5" H 6315 1596 50  0000 L CNN
 F 1 "1uF" H 6315 1505 50  0000 L CNN
-F 2 "Capacitor_SMD:C_0402_1005Metric" H 6238 1400 50  0001 C CNN
+F 2 "Capacitor_SMD:C_0805_2012Metric_Pad1.15x1.40mm_HandSolder" H 6238 1400 50  0001 C CNN
 F 3 "~" H 6200 1550 50  0001 C CNN
 	1    6200 1550
@@
 F 0 "C6" H 6715 1596 50  0000 L CNN
 F 1 "100nF" H 6715 1505 50  0000 L CNN
-F 2 "Capacitor_SMD:C_0402_1005Metric" H 6638 1400 50  0001 C CNN
+F 2 "Capacitor_SMD:C_0805_2012Metric_Pad1.15x1.40mm_HandSolder" H 6638 1400 50  0001 C CNN
 F 3 "~" H 6600 1550 50  0001 C CNN
 	1    6600 1550
@@
 F 0 "C1" H 1715 1746 50  0000 L CNN
 F 1 ".1uF" H 1715 1655 50  0000 L CNN
-F 2 "Capacitor_SMD:C_0402_1005Metric" H 1638 1550 50  0001 C CNN
+F 2 "Capacitor_SMD:C_0805_2012Metric_Pad1.15x1.40mm_HandSolder" H 1638 1550 50  0001 C CNN
 F 3 "~" H 1600 1700 50  0001 C CNN
 	1    1600 1700
@@
 F 0 "R2" V 1143 1300 50  0000 C CNN
 F 1 "10k" V 1234 1300 50  0000 C CNN
-F 2 "Resistor_SMD:R_0402_1005Metric" V 1280 1300 50  0001 C CNN
+F 2 "Resistor_SMD:R_0805_2012Metric_Pad1.15x1.40mm_HandSolder" V 1280 1300 50  0001 C CNN
 F 3 "~" H 1350 1300 50  0001 C CNN
 	1    1350 1300
@@
 F 0 "R1" H 930 954 50  0000 R CNN
 F 1 "10k" H 930 1045 50  0000 R CNN
-F 2 "Resistor_SMD:R_0402_1005Metric" V 930 1000 50  0001 C CNN
+F 2 "Resistor_SMD:R_0805_2012Metric_Pad1.15x1.40mm_HandSolder" V 930 1000 50  0001 C CNN
 F 3 "~" H 1000 1000 50  0001 C CNN
 	1    1000 1000
@@
 F 0 "C4" H 1715 7246 50  0000 L CNN
 F 1 ".1uF" H 1715 7155 50  0000 L CNN
-F 2 "Capacitor_SMD:C_0402_1005Metric" H 1638 7050 50  0001 C CNN
+F 2 "Capacitor_SMD:C_0805_2012Metric_Pad1.15x1.40mm_HandSolder" H 1638 7050 50  0001 C CNN
 F 3 "~" H 1600 7200 50  0001 C CNN
 	1    1600 7200
@@
 F 0 "R8" V 1143 6800 50  0000 C CNN
 F 1 "10k" V 1234 6800 50  0000 C CNN
-F 2 "Resistor_SMD:R_0402_1005Metric" V 1280 6800 50  0001 C CNN
+F 2 "Resistor_SMD:R_0805_2012Metric_Pad1.15x1.40mm_HandSolder" V 1280 6800 50  0001 C CNN
 F 3 "~" H 1350 6800 50  0001 C CNN
 	1    1350 6800
@@
 F 0 "R7" H 930 6454 50  0000 R CNN
 F 1 "10k" H 930 6545 50  0000 R CNN
-F 2 "Resistor_SMD:R_0402_1005Metric" V 930 6500 50  0001 C CNN
+F 2 "Resistor_SMD:R_0805_2012Metric_Pad1.15x1.40mm_HandSolder" V 930 6500 50  0001 C CNN
 F 3 "~" H 1000 6500 50  0001 C CNN
 	1    1000 6500
@@
 F 0 "R6" V 1143 5000 50  0000 C CNN
 F 1 "10k" V 1234 5000 50  0000 C CNN
-F 2 "Resistor_SMD:R_0402_1005Metric" V 1280 5000 50  0001 C CNN
+F 2 "Resistor_SMD:R_0805_2012Metric_Pad1.15x1.40mm_HandSolder" V 1280 5000 50  0001 C CNN
 F 3 "~" H 1350 5000 50  0001 C CNN
 	1    1350 5000
@@
 F 0 "R5" H 930 4654 50  0000 R CNN
 F 1 "10k" H 930 4745 50  0000 R CNN
-F 2 "Resistor_SMD:R_0402_1005Metric" V 930 4700 50  0001 C CNN
+F 2 "Resistor_SMD:R_0805_2012Metric_Pad1.15x1.40mm_HandSolder" V 930 4700 50  0001 C CNN
 F 3 "~" H 1000 4700 50  0001 C CNN
 	1    1000 4700
@@
 F 0 "R4" H 930 2804 50  0000 R CNN
 F 1 "10k" H 930 2895 50  0000 R CNN
-F 2 "Resistor_SMD:R_0402_1005Metric" V 930 2850 50  0001 C CNN
+F 2 "Resistor_SMD:R_0805_2012Metric_Pad1.15x1.40mm_HandSolder" V 930 2850 50  0001 C CNN
 F 3 "~" H 1000 2850 50  0001 C CNN
 	1    1000 2850
@@
 F 0 "R3" V 1143 3150 50  0000 C CNN
 F 1 "10k" V 1234 3150 50  0000 C CNN
-F 2 "Resistor_SMD:R_0402_1005Metric" V 1280 3150 50  0001 C CNN
+F 2 "Resistor_SMD:R_0805_2012Metric_Pad1.15x1.40mm_HandSolder" V 1280 3150 50  0001 C CNN
 F 3 "~" H 1350 3150 50  0001 C CNN
 	1    1350 3150
@@
 F 0 "C2" H 1715 3596 50  0000 L CNN
 F 1 ".1uF" H 1715 3505 50  0000 L CNN
-F 2 "Capacitor_SMD:C_0402_1005Metric" H 1638 3400 50  0001 C CNN
+F 2 "Capacitor_SMD:C_0805_2012Metric_Pad1.15x1.40mm_HandSolder" H 1638 3400 50  0001 C CNN
 F 3 "~" H 1600 3550 50  0001 C CNN
 	1    1600 3550
@@
 F 0 "C3" H 1715 5446 50  0000 L CNN
 F 1 ".1uF" H 1715 5355 50  0000 L CNN
-F 2 "Capacitor_SMD:C_0402_1005Metric" H 1638 5250 50  0001 C CNN
+F 2 "Capacitor_SMD:C_0805_2012Metric_Pad1.15x1.40mm_HandSolder" H 1638 5250 50  0001 C CNN
 F 3 "~" H 1600 5400 50  0001 C CNN
 	1    1600 5400
@@
 F 0 "C7" H 3415 5546 50  0000 L CNN
 F 1 ".1uF" H 3415 5455 50  0000 L CNN
-F 2 "Capacitor_SMD:C_0402_1005Metric" H 3338 5350 50  0001 C CNN
+F 2 "Capacitor_SMD:C_0805_2012Metric_Pad1.15x1.40mm_HandSolder" H 3338 5350 50  0001 C CNN
 F 3 "~" H 3300 5500 50  0001 C CNN
 	1    3300 5500
@@
 F 0 "R9" H 2920 4996 50  0000 L CNN
 F 1 "100k" H 2920 4905 50  0000 L CNN
-F 2 "Resistor_SMD:R_0402_1005Metric" V 2780 4950 50  0001 C CNN
+F 2 "Resistor_SMD:R_0805_2012Metric_Pad1.15x1.40mm_HandSolder" V 2780 4950 50  0001 C CNN
 F 3 "~" H 2850 4950 50  0001 C CNN
 	1    2850 4950
@@
 F 0 "R10" V 2543 1150 50  0000 C CNN
 F 1 "10k" V 2634 1150 50  0000 C CNN
-F 2 "Resistor_SMD:R_0402_1005Metric" V 2680 1150 50  0001 C CNN
+F 2 "Resistor_SMD:R_0805_2012Metric_Pad1.15x1.40mm_HandSolder" V 2680 1150 50  0001 C CNN
 F 3 "~" H 2750 1150 50  0001 C CNN
 	1    2750 1150
@@
 F 0 "C8" H 3015 1996 50  0000 L CNN
 F 1 "1uF" H 3015 1905 50  0000 L CNN
-F 2 "Capacitor_SMD:C_0402_1005Metric" H 2938 1800 50  0001 C CNN
+F 2 "Capacitor_SMD:C_0805_2012Metric_Pad1.15x1.40mm_HandSolder" H 2938 1800 50  0001 C CNN
 F 3 "~" H 2900 1950 50  0001 C CNN
 	1    2900 1950
@@
 F 0 "R11" V 2543 1500 50  0000 C CNN
 F 1 "510" V 2634 1500 50  0000 C CNN
-F 2 "Resistor_SMD:R_0402_1005Metric" V 2680 1500 50  0001 C CNN
+F 2 "Resistor_SMD:R_0805_2012Metric_Pad1.15x1.40mm_HandSolder" V 2680 1500 50  0001 C CNN
 F 3 "~" H 2750 1500 50  0001 C CNN
 	1    2750 1500
