File: ECE477/ECE477.sch (KiCad schematic (older format))
At the start: 3 parts

Commit message: Testing
Testing
Parts:
- added C1: 4.7uF, symbol pspice:CAP
- added C10, C11, C12, C13, C14, C15, C17, C19, C2, C3, C4, C5, C6, C7, C8, C9: 100nF, symbol pspice:CAP
- added C16, C18: 1uF, symbol pspice:CAP
- added IC1: PTN78020WAH, EUL(R-PDSS-B7), symbol SamacSys_Parts:PTN78020WAH
- added PS1: R-555.0DA, CONV_R-555.0DA, symbol R-555.0DA:R-555.0DA
- added R1, R2: 0R, symbol Device:R_US
- added U2: BQ29312APW, PW24, symbol 2020-09-16_23-09-37:BQ29312APW
- gave numbers to parts that had none: 1
Connections:
- net VCAP: now reaches U1.103 (VCAP)
- net VCAP: now also U1.140 (VCAP), U1.68 (VCAP)
- net GND: now reaches U1.104 (VSS)
- net GND: now also U1.118 (VSS), U1.12 (VSS), U1.128 (VSS), U1.141 (VSS), U1.18 (VSS), U1.33 (VSS), U1.41 (VSS), U1.55 (VSS), U1.6 (VSS), U1.69 (VSS), U1.8 (VBAT), U1.80 (VSS), U1.89 (VSS), C1.2, C10.2, C11.2, C12.2, C13.2, C14.2, C15.2, C2.2, C3.2, C4.2, C5.2, C6.2, C7.2, C8.2, C9.2
- net VDD_LDO: now reaches U1.105 (VDDLDO)
- net VDD_LDO: now also U1.143 (VDDLDO), U1.70 (VDDLDO)
- net VDD_MCU: now reaches U1.106 (VDD)
- net VDD_MCU: now also U1.119 (VDD), U1.129 (VDD), U1.13 (VDD), U1.144 (VDD), U1.19 (VDD), U1.32 (VDD), U1.42 (VDD), U1.56 (VDD), U1.7 (VDD), U1.71 (VDD), U1.79 (VDD), U1.92 (VDD), C1.1, C10.1, C11.1, C12.1, C13.1, C14.1, C2.1, C3.1, C4.1, C5.1, C6.1, C7.1, C8.1, C9.1, R1.1
- net VREF+: now reaches U1.35 (VREF+)
- net VREF+: now also C18.1, C19.1, R2.2
- net VDDA: now reaches U1.36 (VDDA)
- net VDDA: now also C16.1, C17.1, R1.2, R2.1
- new net: PS1.10 (VOUT), PS1.9 (VOUT)
- new net: PS1.2 (VIN), PS1.3 (VIN), PS1.4 (VIN)
- new net: PS1.5 (GND), PS1.6 (GND), PS1.7 (GND), PS1.8 (GND)
- new net GNDA: C16.2, C17.2, C18.2, C19.2
- new net VBAT: C15.1
Other:
- moved on the sheet: U1A, U1B, U1C

Commit message: Added 4 LED pads
Added 4 cirucits for the installation of LEDs still need to calculate the resitance to apply to the LEDs based on colors
Parts:
- added Q? (x4): NPN SOT23, digikey-footprints:SOT-23-3, symbol dk_Transistors-Bipolar-BJT-Single:MMBT2222ALT1G
- added R? (x4): 100K, symbol Device:R_US
- added R? (x4): 47K, symbol Device:R_US
Connections:
- net GND: now also Q?.2 (E), Q?.2 (E), Q?.2 (E), Q?.2 (E), R?.1, R?.1, R?.1, R?.1
- new net: Q?.1 (B), R?.2, R?.2 (x4)
Other:
- moved on the sheet: C1, C10, C11, C12, C13, C14, C15, C16, C17, C18, C19, C2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
